Commit message: Update panda.urdf
dea

File: deps/Panda/panda.urdf (robot description, URDF)
Before this commit: robot panda, 12 links, 11 joints
Links:
- link panda_hand: geometry collision mesh filename=package://Panda/meshes/collision/hand.obj; visual mesh filename=package://Panda/meshes/visual/hand.dae
- link panda_leftfinger: geometry collision mesh filename=package://Panda/meshes/collision/finger.obj; visual mesh filename=package://Panda/meshes/visual/finger.dae
- link panda_link0: geometry collision mesh filename=package://Panda/meshes/collision/link0.obj; visual mesh filename=package://Panda/meshes/visual/link0.dae
- link panda_link1: geometry collision mesh filename=package://Panda/meshes/collision/link1.obj; visual mesh filename=package://Panda/meshes/visual/link1.dae
- link panda_link2: geometry collision mesh filename=package://Panda/meshes/collision/link2.obj; visual mesh filename=package://Panda/meshes/visual/link2.dae
- link panda_link3: geometry collision mesh filename=package://Panda/meshes/collision/link3.obj; visual mesh filename=package://Panda/meshes/visual/link3.dae
- link panda_link4: geometry collision mesh filename=package://Panda/meshes/collision/link4.obj; visual mesh filename=package://Panda/meshes/visual/link4.dae
- link panda_link5: geometry collision mesh filename=package://Panda/meshes/collision/link5.obj; visual mesh filename=package://Panda/meshes/visual/link5.dae
- link panda_link6: geometry collision mesh filename=package://Panda/meshes/collision/link6.obj; visual mesh filename=package://Panda/meshes/visual/link6.dae
- link panda_link7: geometry collision mesh filename=package://Panda/meshes/collision/link7.obj; visual mesh filename=package://Panda/meshes/visual/link7.dae
- link panda_rightfinger: geometry collision mesh filename=package://Panda/meshes/collision/finger.obj; visual mesh filename=package://Panda/meshes/visual/finger.dae
